File: UKey_STM32.sch (KiCad schematic (older format))
At the start: 22 parts, among them J1 USB_A, J2 Conn_01x04_Male, SW1 SW_Push, SW2 SW_DIP_x02, U1 NUF2221W1, U2 LDK130-33_SOT23_SOT353, U3 M25PX32-VMW, U4 STM32F103C8Tx, Y1 Crystal_GND24

Commit message: Fixed LDO EN Pin.
Connections:
- net VBUS: now also U2.3 (EN)
Changed lines of the file:
@@
 Connection ~ 2300 1000
 Wire Wire Line
-	1300 1100 1200 1100
-Wire Wire Line
-	1200 1100 1200 1350
+	850  1100 1300 1100
 Wire Wire Line
 	1050 2850 1050 3100
@@
 Wire Wire Line
 	5100 4550 4900 4550
+Connection ~ 850  1100
 $EndSCHEMATC

Commit message: Updated board.
Parts:
- SW2: footprint Buttons_Switches_SMD:SW_DIP_x2_W5.08mm_Slide_Copal_CHS-A -> Buttons_Switches_SMD:SW_DIP_x2_W7.62mm_Slide_Copal_CHS-B
- U1: footprint TO_SOT_Packages_SMD:SOT-23-6_Handsoldering -> TO_SOT_Packages_SMD:SOT-363_SC-70-6_Handsoldering
Connections:
- net EMI_DM: now also U1.4 (D2c); no longer U1.6 (D1c)
- net EMI_DP: now also U1.6 (D1c); no longer U1.4 (D2c)
- net USB_DM: now also U1.3 (D2i); no longer U1.1 (D1i)
- net USB_DP: now also U1.1 (D1i); no longer U1.3 (D2i)
Changed lines of the file:
@@
 	1    0    0    -1
 $EndComp
+Text GLabel 1250 4550 0    60   Input ~ 0
+USB_DP
 Text GLabel 1250 4750 0    60   Input ~ 0
-USB_DP
-Text GLabel 1250 4550 0    60   Input ~ 0
 USB_DM
 $Comp
@@
 F 0 "SW2" H 1550 6350 50  0000 C CNN
 F 1 "SW_DIP_x02" H 1550 5950 50  0000 C CNN
-F 2 "Buttons_Switches_SMD:SW_DIP_x2_W5.08mm_Slide_Copal_CHS-A" H 1550 6100 50  0001 C CNN
+F 2 "Buttons_Switches_SMD:SW_DIP_x2_W7.62mm_Slide_Copal_CHS-B" H 1550 6100 50  0001 C CNN
 F 3 "" H 1550 6100 50  0001 C CNN
 	1    1550 6100
@@
 F 0 "U1" H 1550 4850 70  0000 C CNN
 F 1 "NUF2221W1" H 1750 4425 70  0000 C CNN
-F 2 "TO_SOT_Packages_SMD:SOT-23-6_Handsoldering" H 1750 4650 60  0001 C CNN
+F 2 "TO_SOT_Packages_SMD:SOT-363_SC-70-6_Handsoldering" H 1750 4650 60  0001 C CNN
 F 3 "" H 1750 4650 60  0001 C CNN
 	1    1750 4650
@@
 Text GLabel 1500 7350 2    60   Input ~ 0
 EMI_DP
+Text GLabel 2250 4750 2    60   Input ~ 0
+EMI_DM
 Text GLabel 2250 4550 2    60   Input ~ 0
-EMI_DM
-Text GLabel 2250 4750 2    60   Input ~ 0
 EMI_DP
 $Comp
